File: MotorDriver.kicad_sch (KiCad schematic)
At the start: 18 parts, among them IC1 TMC2209-LA or HR4988E, J6 Conn_01x03_Pin, J8 Conn_01x06_Pin

Commit message: fix work for piezo and step driver
Parts:
- added R38: 10k, piezo_driver:R_0603_1608Metric_u, symbol piezo_driver:R
- R70, R71: value 0 -> 1; LCSC C21189 -> C22936
Connections:
- net +3V3: now also R21.1, R38.1
- net SPREAD: now also IC1.11 (DIAG); no longer R21.1
- net at IC1.12 (INDEX): now also R38.2
- no-connect marks 5 -> 3
